Commit message: RTAB-Map added

File: ros/simulation/urdf/hermes2.xacro (robot description, xacro)
@@ -1,4 +1,5 @@
 <?xml version="1.0" ?>
-<robot name="hermes">
+<robot name="my_vehicle">
+  <!-- RGBD Camera-->
   <link name="base_link">
     <inertial>
@@ -160,11 +161,5 @@
     <origin rpy="-1.5708 0 0" xyz="0.159795 0.3005 -.38978" />
   </joint>
-  <link name = "camera_center"/>
-  <joint name = "camera_center_base_link" type = "fixed">
-    <origin xyz="0.630975 0.0 -0.1807467" rpy="0 0 0" />
-    <parent link="base_link" />
-    <child link="camera_center" />
-  </joint>
-  <link name="camera_link_left">
+  <link name="lidar_link">
     <collision>
       <origin xyz="0 0 0" rpy="0 0 0" />
@@ -185,62 +180,57 @@
     </inertial>
   </link>
-  <joint name="camera_joint_left" type="fixed">
-    <origin xyz="0.0 0.1 0.0" rpy="0 0 0" />
-    <parent link="camera_center" />
-    <child link="camera_link_left" />
-  </joint>
-    <link name="camera_link_right">
-    <collision>
-      <origin xyz="0 0 0" rpy="0 0 0" />
+  <joint name="lidar_joint" type="fixed">
+    <origin xyz="0.630975 0 -0.1807467" rpy="0 0 0" />
+    <parent link="base_link" />
+    <child link="lidar_link" />
+  </joint>
+  <link name="camera_link">
+    <visual>
+      <origin rpy="0 0 0" xyz="0 0 0" />
+      <geometry>
+        <box size="0.05 0.05 0.05" />
+      </geometry>
+      <material name="Blue" />
+    </visual>
+  </link>
+  <joint name="camera_joint" type="fixed">
+    <origin rpy="0 1.0466 0" xyz="0.555975 0 0.72404" />
+    <parent link="base_link" />
+    <child link="camera_link" />
+  </joint>
+  <joint name="camera_optical_joint" type="fixed">
+    <origin xyz="0 0 0" rpy="-1.5707 0 -1.5707"/>
+    <parent link="camera_link"/>
+    <child link="camera_link_optical"/>
+  </joint>
+  <link name="camera_link_optical">
+  </link>
+  <link name="imu_link">
+    <visual>
+      <origin rpy="0 0 0" xyz="0 0 0" />
+      <geometry>
+        <box size="0.05 0.05 0.05" />
+      </geometry>
+      <material name="Blue" />
+    </visual>
+  </link>
+  <joint name="imu_joint" type="fixed">
+    <origin rpy="0 0 0" xyz="0.16 0 0" />
+    <parent link="base_link" />
+    <child link="imu_link" />
+  </joint>
+  <link name="gps_link">
+    <visual>
+      <origin rpy="0 0 0" xyz="0 0 0" />
       <geometry>
         <box size="0.1 0.1 0.1" />
       </geometry>
-    </collision>
-    <visual>
-      <origin xyz="0 0 0" rpy="0 0 0" />
-      <geometry>
-        <box size="0.1 0.1 0.1" />
-      </geometry>
-    </visual>
-    <inertial>
-      <mass value="1e-5" />
-      <origin xyz="0 0 0" rpy="0 0 0" />
-      <inertia ixx="1e-6" ixy="0" ixz="0" iyy="1e-6" iyz="0" izz="1e-6" />
-    </inertial>
-  </link>
-  <joint name="camera_joint_right" type="fixed">
-    <origin xyz="0.0 -0.1 0.0" rpy="0 0 0" />
-    <parent link="camera_center" />
-    <child link="camera_link_right" />
-  </joint>
-  <link name="left_camera_optical_frame"/>
-  <joint name="left_camera_optical_frame_joint" type="fixed">
-    <origin xyz="0 0 0" rpy="0.0 0.0 0.0" />
-    <parent link="camera_link_left" />
-    <child link="left_camera_optical_frame"/>
-  </joint>
-  <link name="lidar_link">
-    <collision>
-      <origin xyz="0 0 0" rpy="0 0 0" />
-      <geometry>
-        <box size="0.1 0.1 0.1" />
-      </geometry>
-    </collision>
-    <visual>
-      <origin xyz="0 0 0" rpy="0 0 0" />
-      <geometry>
-        <box size="0.1 0.1 0.1" />
-      </geometry>
-    </visual>
-    <inertial>
-      <mass value="1e-5" />
-      <origin xyz="0 0 0" rpy="0 0 0" />
-      <inertia ixx="1e-6" ixy="0" ixz="0" iyy="1e-6" iyz="0" izz="1e-6" />
-    </inertial>
-  </link>
-  <joint name="lidar_joint" type="fixed">
-    <origin xyz="0.630975 0 0.3807467" rpy="0 0 0" />
-    <parent link="base_link" />
-    <child link="lidar_link" />
+      <material name="Blue" />
+    </visual>
+  </link>
+  <joint name="gps_joint" type="fixed">
+    <origin rpy="0 0 0" xyz="0.16 0 0.48011" />
+    <parent link="base_link" />
+    <child link="gps_link" />
   </joint>
   <gazebo>
@@ -287,11 +277,10 @@
       </ray>
       <plugin filename="libgazebo_ros_laser.so" name="gazebo_ros_head_hokuyo_controller">
-        <topicName>/scan</topicName>
+        <topicName>scan</topicName>
         <frameName>lidar_link</frameName>
       </plugin>
     </sensor>
   </gazebo>
-  <!--
-  <gazebo reference="camera_link">
+  <!-- <gazebo reference="camera_link">
     <sensor type="camera" name="camera1">
       <update_rate>30.0</update_rate>
@@ -328,60 +317,81 @@
       </plugin>
     </sensor>
-  </gazebo>
--->
-  <!--stereo camera config-->
-  <gazebo reference="camera_center">
-    <sensor type="multicamera" name="stereo_camera">
-      <update_rate>30.0</update_rate>
-      <camera name="left">
-        <horizontal_fov>1.3962634</horizontal_fov>
-        <image>
-          <width>800</width>
-          <height>800</height>
-          <format>R8G8B8</format>
-        </image>
-        <clip>
-          <near>0.02</near>
-          <far>300</far>
-        </clip>
-        <noise>
-          <type>gaussian</type>
-          <mean>0.0</mean>
-          <stddev>0.007</stddev>
-        </noise>
-      </camera>
-      <camera name="right">
-        <pose>0 -0.07 0 0 0 0</pose>
-        <horizontal_fov>1.3962634</horizontal_fov>
-        <image>
-          <width>800</width>
-          <height>800</height>
-          <format>R8G8B8</format>
-        </image>
-        <clip>
-          <near>0.02</near>
-          <far>300</far>
-        </clip>
-        <noise>
-          <type>gaussian</type>
-          <mean>0.0</mean>
-          <stddev>0.007</stddev>
-        </noise>
-      </camera>
-      <plugin name="stereo_camera_controller" filename="libgazebo_ros_multicamera.so">
-        <alwaysOn>true</alwaysOn>
-        <updateRate>0.0</updateRate>
-        <cameraName>stereo_camera</cameraName>
-        <imageTopicName>image_raw</imageTopicName>
-        <cameraInfoTopicName>camera_info</cameraInfoTopicName>
-        <frameName>left_camera_optical_frame</frameName>
-        <!--<rightFrameName>right_camera_optical_frame</rightFrameName>-->
-        <hackBaseline>0.07</hackBaseline>
-        <distortionK1>0.0</distortionK1>
-        <distortionK2>0.0</distortionK2>
-        <distortionK3>0.0</distortionK3>
-        <distortionT1>0.0</distortionT1>
-        <distortionT2>0.0</distortionT2>
+  </gazebo> -->
+  <!-- RGBD Camera -->
+  <gazebo reference="camera_link">
+    <sensor type="depth" name="camera1">
+        <always_on>1</always_on>
+        <update_rate>20.0</update_rate>
+        <visualize>true</visualize>
+        <camera>
+            <horizontal_fov>1.047</horizontal_fov>
+            <image>
+                <width>640</width>
+                <height>480</height>
+                <format>R8G8B8</format>
+            </image>
+            <depth_camera>
+            </depth_camera>
+            <clip>
+                <near>0.1</near>
+                <far>20</far>
+            </clip>
+        </camera>
+             <plugin name="camera_controller" filename="libgazebo_ros_openni_kinect.so">
+             <alwaysOn>true</alwaysOn>
+                <updateRate>10.0</updateRate>
+                <cameraName>camera</cameraName>
+                <frameName>camera_link_optical</frameName>
+            <imageTopicName>rgb/image_raw</imageTopicName>
+            <depthImageTopicName>depth/image_raw</depthImageTopicName>
+            <pointCloudTopicName>depth/points</pointCloudTopicName>
+            <cameraInfoTopicName>rgb/camera_info</cameraInfoTopicName>
+            <depthImageCameraInfoTopicName>depth/camera_info</depthImageCameraInfoTopicName>
+            <pointCloudCutoff>0.4</pointCloudCutoff>
+                <hackBaseline>0.07</hackBaseline>
+                <distortionK1>0.0</distortionK1>
+                <distortionK2>0.0</distortionK2>
+                <distortionK3>0.0</distortionK3>
+                <distortionT1>0.0</distortionT1>
+                <distortionT2>0.0</distortionT2>
+            <CxPrime>0.0</CxPrime>
+            <Cx>0.0</Cx>
+            <Cy>0.0</Cy>
+            <focalLength>0.0</focalLength>
+            </plugin>
+    </sensor>
+  </gazebo>
+  <!-- gps-->
+  <gazebo>
+    <plugin name="novatel_gps_sim" filename="libhector_gazebo_ros_gps.so">
+      <alwaysOn>1</alwaysOn>
+      <updateRate>10.0</updateRate>
+      <bodyName>gps_link</bodyName>
+      <topicName>gps</topicName>
+      <velocityTopicName>gps_velocity</velocityTopicName>
+      <drift>5.0 5.0 5.0</drift>
+      <gaussianNoise>0.1 0.1 0.1</gaussianNoise>
+      <velocityDrift>0 0 0</velocityDrift>
+      <velocityGaussianNoise>0.1 0.1 0.1</velocityGaussianNoise>
+    </plugin>
+  </gazebo>
+  <!-- imu -->
+  <gazebo reference="imu_link">
+    <gravity>true</gravity>
+    <sensor name="imu_sensor" type="imu">
+      <always_on>true</always_on>
+      <update_rate>100.0</update_rate>
+      <visualize>false</visualize>
+      <topic>imu</topic>
+      <plugin filename="libgazebo_ros_imu_sensor.so" name="imu_plugin">
+        <topicName>imu</topicName>
+        <bodyName>imu_link</bodyName>
+        <updateRateHZ>100.0</updateRateHZ>
+        <gaussianNoise>0.0</gaussianNoise>
+        <xyzOffset>0 0 0</xyzOffset>
+        <rpyOffset>0 0 0</rpyOffset>
+        <frameName>imu_link</frameName>
       </plugin>
+      <pose>0 0 0 0 0 0</pose>
     </sensor>
   </gazebo>
